File: PCB/easyPICO WiFi.kicad_pcb (KiCad board)
At the start: 2 copper layers, 41 x 62 mm, 36 parts, among them J1 USB_C_Receptacle_USB2.0_14P, J2 Conn_01x20, J3 1x3, J4 Conn_01x20, J5 Conn_01x01, SW1 SW_Push, U1 2040, U2 MCP, U3 Mem, Y1 12 MHz

Commit message: add files
Parts:
- moved G*** 22.8 mm to (145.9, 117.2)
- moved G*** 9.31 mm to (123.9, 99.8), turned to -90 degrees
Routing:
- net QSPI_SD1: track 26.0 -> 15.7 mm
- net GND: track 287.3 -> 283.7 mm
- net +3V3: track 138.5 -> 136.3 mm
- added copper zone on B.Cu, net GND
- added copper zone on F.Cu, net GND
Other:
- board text added: "@chicken"
- board text added: "X"
- board text removed: "GPIOs 26, 27, 28, and 29 are all ADC pins."
- board text removed: "The"
- board text removed: "easyPi WiFi"
